File: Solar-Cell-Holder.sch (KiCad schematic (older format))
At the start: 3 parts, among them J1 Conn_01x01_Female, J2 Conn_01x01_Female, U1 XTJ

Commit message: finished
Parts:
- removed J1, J2: Conn_01x01_Female, Connector_PinSocket_2.00mm:PinSocket_1x01_P2.00mm_Vertical, symbol Connector:Conn_01x01_Female
- added J1, J2: Conn_01x02_Female, Connector_PinSocket_2.00mm:PinSocket_1x02_P2.00mm_Vertical, symbol Connector:Conn_01x02_Female
- U1: symbol XTJ:XTJ -> Solar-Cell-Holder-rescue:XTJ-XTJ
Connections:
- net at U1.~ (Positive): now also J2.1 (Pin_1), J2.2 (Pin_2)
- new net: J1.1 (Pin_1), J1.2 (Pin_2), U1.~ (Positive)
Changed lines of the file:
@@
 EESchema Schematic File Version 4
+LIBS:Solar-Cell-Holder-cache
 EELAYER 29 0
 EELAYER END
@@
 $EndDescr
 $Comp
-L XTJ:XTJ U1
+L Solar-Cell-Holder-rescue:XTJ-XTJ U1
 U 1 1 5DD79E02
 P 4700 3850
@@
 Wire Wire Line
 	4650 4150 4750 4150
+Wire Wire Line
+	4650 4150 4650 4350
 $Comp
-L Connector:Conn_01x01_Female J1
-U 1 1 5DD7A3A1
-P 4650 4550
-F 0 "J1" V 4496 4598 50  0000 L CNN
-F 1 "Conn_01x01_Female" V 4587 4598 50  0000 L CNN
-F 2 "Connector_PinSocket_2.00mm:PinSocket_1x01_P2.00mm_Vertical" H 4650 4550 50  0001 C CNN
-F 3 "~" H 4650 4550 50  0001 C CNN
-	1    4650 4550
+L Connector:Conn_01x02_Female J1
+U 1 1 5DD86995
+P 4700 4550
+F 0 "J1" V 4546 4598 50  0000 L CNN
+F 1 "Conn_01x02_Female" V 4637 4598 50  0000 L CNN
+F 2 "Connector_PinSocket_2.00mm:PinSocket_1x02_P2.00mm_Vertical" H 4700 4550 50  0001 C CNN
+F 3 "~" H 4700 4550 50  0001 C CNN
+	1    4700 4550
 	0    1    1    0
 $EndComp
+Wire Wire Line
+	4600 4350 4650 4350
+Connection ~ 4650 4350
+Wire Wire Line
+	4650 4350 4700 4350
 $Comp
-L Connector:Conn_01x01_Female J2
-U 1 1 5DD7C4F1
-P 5350 4350
-F 0 "J2" V 5196 4398 50  0000 L CNN
-F 1 "Conn_01x01_Female" V 5287 4398 50  0000 L CNN
-F 2 "Connector_PinSocket_2.00mm:PinSocket_1x01_P2.00mm_Vertical" H 5350 4350 50  0001 C CNN
-F 3 "~" H 5350 4350 50  0001 C CNN
-	1    5350 4350
+L Connector:Conn_01x02_Female J2
+U 1 1 5DD87EAB
+P 5300 4200
+F 0 "J2" V 5146 4248 50  0000 L CNN
+F 1 "Conn_01x02_Female" V 5237 4248 50  0000 L CNN
+F 2 "Connector_PinSocket_2.00mm:PinSocket_1x02_P2.00mm_Vertical" H 5300 4200 50  0001 C CNN
+F 3 "~" H 5300 4200 50  0001 C CNN
+	1    5300 4200
 	1    0    0    -1
 $EndComp
 Wire Wire Line
-	4900 4150 4900 4350
+	5100 4200 5100 4250
 Wire Wire Line
-	4900 4350 5150 4350
+	5100 4250 4900 4250
 Wire Wire Line
-	4650 4150 4650 4350
+	4900 4250 4900 4150
+Connection ~ 5100 4250
+Wire Wire Line
+	5100 4250 5100 4300
 $EndSCHEMATC
